Commit message: Add robotiq_2f_140 gripper

File: grab2_controller/description/panda/panda.urdf.xacro (robot description, xacro)
@@ -1,5 +1,5 @@
 <?xml version="1.0"?>
 <robot xmlns:xacro="http://www.ros.org/wiki/xacro" name="panda">
-    <xacro:arg name="initial_positions_file" default="initial_positions.yaml" />
+    <xacro:arg name="initial_positions_file" default="$(find grab2_controller)/config/panda/initial_positions.yaml" />
     <xacro:arg name="ros2_control_hardware_type" default="mock_components" />
     <!-- Import panda urdf file -->

File: grab2_controller/description/ur/ur.ros2_control.xacro (robot description, xacro)
@@ -1,5 +1,5 @@
 <?xml version="1.0"?>
 <robot xmlns:xacro="http://www.ros.org/wiki/xacro">
-    <xacro:macro name="ur_ros2_control" params="name initial_positions_file ros2_control_hardware_type">
+    <xacro:macro name="ur_ros2_control" params="name initial_positions_file ros2_control_hardware_type use_gripper">
         <xacro:property name="initial_positions" value="${xacro.load_yaml(initial_positions_file)['initial_positions']}"/>
         <ros2_control name="${name}" type="system">
@@ -68,4 +68,12 @@
                 </state_interface>
             </joint>
+            <!-- Robotiq Gripper -->
+            <xacro:if value="${use_gripper}">
+              <joint name="finger_joint">
+                <command_interface name="position"/>
+                <state_interface name="position"/>
+                <state_interface name="velocity"/>
+              </joint>
+            </xacro:if>
         </ros2_control>
     </xacro:macro>

File: grab2_controller/description/ur/ur.urdf.xacro (robot description, xacro)
@@ -1,5 +1,5 @@
 <?xml version="1.0"?>
-<robot xmlns:xacro="http://www.ros.org/wiki/xacro" name="ur10e">
-    <xacro:arg name="initial_positions_file" default="initial_positions.yaml" />
+<robot xmlns:xacro="http://www.ros.org/wiki/xacro" name="ur">
+    <xacro:arg name="initial_positions_file" default="$(find grab2_controller)/config/ur/initial_positions.yaml" />
     <xacro:arg name="ros2_control_hardware_type" default="mock_components" />
     <!-- parameters -->
@@ -10,4 +10,5 @@
     <xacro:arg name="physical_params" default="$(find ur_description)/config/$(arg ur_type)/physical_parameters.yaml"/>
     <xacro:arg name="visual_params" default="$(find ur_description)/config/$(arg ur_type)/visual_parameters.yaml"/>
+    <xacro:arg name="use_robotiq_gripper" default="false"/>
     <!-- arm -->
     <!-- <Modified from filename="$(find ur_description)/urdf/ur.urdf.xacro"/> -->
@@ -27,6 +28,10 @@
     <!-- create link fixed to the "world" -->
    <link name="world" />
-    <!-- Import ur10e ros2_control description -->
-    <xacro:include filename="ur10e.ros2_control.xacro" />
-    <xacro:ur_ros2_control name="URFakeSystem" initial_positions_file="$(arg initial_positions_file)" ros2_control_hardware_type="$(arg ros2_control_hardware_type)"/>
+    <!-- Import ros2_control description -->
+    <xacro:include filename="ur.ros2_control.xacro" />
+    <xacro:ur_ros2_control name="URFakeSystem" initial_positions_file="$(arg initial_positions_file)" ros2_control_hardware_type="$(arg ros2_control_hardware_type)" use_gripper="$(arg use_robotiq_gripper)"/>
+    <!-- Robotiq Gripper -->
+    <xacro:if value="$(arg use_robotiq_gripper)">
+        <xacro:include filename="$(find grab2_controller)/description/robotiq_2f_140/robotiq_2f_140.xacro"/>
+    </xacro:if>
 </robot>
