Commit message: sinle thread with no time optimization

File: install/grab2_controller/share/grab2_controller/description/ur/ur.ros2_control.xacro (robot description, xacro)
@@ -1 +1,80 @@
-/home/zaynap/grab/grab2/grab2_controller/description/ur/ur.ros2_control.xacro
+<?xml version="1.0"?>
+<robot xmlns:xacro="http://www.ros.org/wiki/xacro">
+    <xacro:macro name="ur_ros2_control" params="name initial_positions_file ros2_control_hardware_type use_gripper">
+        <xacro:property name="initial_positions" value="${xacro.load_yaml(initial_positions_file)['initial_positions']}"/>
+        <ros2_control name="${name}" type="system">
+            <hardware>
+                <xacro:if value="${ros2_control_hardware_type == 'mock_components'}">
+                    <plugin>mock_components/GenericSystem</plugin>
+                </xacro:if>
+                <xacro:if value="${ros2_control_hardware_type == 'isaac'}">
+                    <plugin>topic_based_ros2_control/TopicBasedSystem</plugin>
+                    <param name="joint_commands_topic">/isaac_joint_commands</param>
+                    <param name="joint_states_topic">/isaac_joint_states</param>
+                </xacro:if>
+            </hardware>
+            <joint name="shoulder_pan_joint">
+                <command_interface name="position"/>
+                <state_interface name="position">
+                  <param name="initial_value">${initial_positions['shoulder_pan_joint']}</param>
+                </state_interface>
+                <state_interface name="velocity">
+                  <param name="initial_value">0.0</param>
+                </state_interface>
+            </joint>
+            <joint name="shoulder_lift_joint">
+                <command_interface name="position"/>
+                <state_interface name="position">
+                  <param name="initial_value">${initial_positions['shoulder_lift_joint']}</param>
+                </state_interface>
+                <state_interface name="velocity">
+                  <param name="initial_value">0.0</param>
+                </state_interface>
+            </joint>
+            <joint name="elbow_joint">
+                <command_interface name="position"/>
+                <state_interface name="position">
+                  <param name="initial_value">${initial_positions['elbow_joint']}</param>
+                </state_interface>
+                <state_interface name="velocity">
+                  <param name="initial_value">0.0</param>
+                </state_interface>
+            </joint>
+            <joint name="wrist_1_joint">
+                <command_interface name="position"/>
+                <state_interface name="position">
+                  <param name="initial_value">${initial_positions['wrist_1_joint']}</param>
+                </state_interface>
+                <state_interface name="velocity">
+                  <param name="initial_value">0.0</param>
+                </state_interface>
+            </joint>
+            <joint name="wrist_2_joint">
+                <command_interface name="position"/>
+                <state_interface name="position">
+                  <param name="initial_value">${initial_positions['wrist_2_joint']}</param>
+                </state_interface>
+                <state_interface name="velocity">
+                  <param name="initial_value">0.0</param>
+                </state_interface>
+            </joint>
+            <joint name="wrist_3_joint">
+                <command_interface name="position"/>
+                <state_interface name="position">
+                  <param name="initial_value">${initial_positions['wrist_3_joint']}</param>
+                </state_interface>
+                <state_interface name="velocity">
+                  <param name="initial_value">0.0</param>
+                </state_interface>
+            </joint>
+            <!-- Robotiq Gripper -->
+            <xacro:if value="${use_gripper}">
+              <joint name="finger_joint">
+                <command_interface name="position"/>
+                <state_interface name="position"/>
+                <state_interface name="velocity"/>
+              </joint>
+            </xacro:if>
+        </ros2_control>
+    </xacro:macro>
+</robot>

File: install/grab2_controller/share/grab2_controller/description/ur/ur.urdf.xacro (robot description, xacro)
@@ -1 +1,37 @@
-/home/zaynap/grab/grab2/grab2_controller/description/ur/ur.urdf.xacro
+<?xml version="1.0"?>
+<robot xmlns:xacro="http://www.ros.org/wiki/xacro" name="ur">
+    <xacro:arg name="initial_positions_file" default="$(find grab2_controller)/config/ur/initial_positions.yaml" />
+    <xacro:arg name="ros2_control_hardware_type" default="mock_components" />
+    <!-- parameters -->
+    <xacro:arg name="name" default="ur10e"/>
+    <xacro:arg name="ur_type" default="ur10e"/>
+    <xacro:arg name="joint_limit_params" default="$(find ur_description)/config/$(arg ur_type)/joint_limits.yaml"/>
+    <xacro:arg name="kinematics_params" default="$(find ur_description)/config/$(arg ur_type)/default_kinematics.yaml"/>
+    <xacro:arg name="physical_params" default="$(find ur_description)/config/$(arg ur_type)/physical_parameters.yaml"/>
+    <xacro:arg name="visual_params" default="$(find ur_description)/config/$(arg ur_type)/visual_parameters.yaml"/>
+    <xacro:arg name="use_robotiq_gripper" default="false"/>
+    <!-- arm -->
+    <!-- <Modified from filename="$(find ur_description)/urdf/ur.urdf.xacro"/> -->
+    <xacro:include filename="$(find ur_description)/urdf/ur_macro.xacro"/>
+    <!-- In ROS2 Humble, Add (generate_ros2_control_tag="false") to the following macro -->
+    <xacro:ur_robot
+        name="$(arg name)"
+        tf_prefix=""
+        parent="world"
+        joint_limits_parameters_file="$(arg joint_limit_params)"
+        kinematics_parameters_file="$(arg kinematics_params)"
+        physical_parameters_file="$(arg physical_params)"
+        visual_parameters_file="$(arg visual_params)"
+        >
+        <origin xyz="0 0 0" rpy="0 0 0" />          <!-- position robot in the world -->
+    </xacro:ur_robot>
+    <!-- create link fixed to the "world" -->
+   <link name="world" />
+    <!-- Import ros2_control description -->
+    <xacro:include filename="ur.ros2_control.xacro" />
+    <xacro:ur_ros2_control name="URFakeSystem" initial_positions_file="$(arg initial_positions_file)" ros2_control_hardware_type="$(arg ros2_control_hardware_type)" use_gripper="$(arg use_robotiq_gripper)"/>
+    <!-- Robotiq Gripper -->
+    <xacro:if value="$(arg use_robotiq_gripper)">
+        <xacro:include filename="$(find grab2_controller)/description/robotiq_2f_140/robotiq_2f_140.xacro"/>
+    </xacro:if>
+</robot>
